File: hardware/controller.sch (KiCad schematic (older format))
At the start: 59 parts, among them J1 USB_B_Micro, J10 Conn_01x05_Male, J11 Conn_01x05_Male, J12 Conn_01x05_Male, J13 Conn_01x05_Male, J14 Conn_01x05_Male, J15 Conn_01x05_Male, J16 Conn_01x05_Male, J17 Conn_01x05_Male, J18 Conn_01x05_Male, J2 AVR-ISP-6, J3 Conn_01x05_Male, J4 Conn_01x05_Male, J5 Conn_01x05_Male, J6 Conn_01x05_Male, J7 Conn_01x05_Male, J8 Conn_01x05_Male, J9 Conn_01x05_Male, Q1 AO3402, Q10 AO3402, Q11 AO3402, Q12 AO3402, Q13 AO3402, Q14 AO3402, Q15 AO3402, Q16 AO3402, Q2 AO3402, Q3 AO3402, Q4 AO3402, Q5 AO3402, Q6 AO3402, Q7 AO3402, Q8 AO3402, Q9 AO3402, U1 CH340C, U2 PCA9685PW, U3 MCP23017_SS, U4 ATmega328P-AU, Y1 14.7456 Mhz

Commit message: fix polyfuse rating
Parts:
- F1: value 750mA -> 350mA
Changed lines of the file:
@@
 P 1850 1750
 F 0 "F1" V 1625 1750 50  0000 C CNN
-F 1 "750mA" V 1716 1750 50  0000 C CNN
+F 1 "350mA" V 1716 1750 50  0000 C CNN
 F 2 "Fuse:Fuse_0805_2012Metric" H 1900 1550 50  0001 L CNN
 F 3 "~" H 1850 1750 50  0001 C CNN
